Commit message: + rviz launch file

File: visualisation/urdf/qolo.urdf (robot description, URDF)
Before this commit: robot qolo, 4 links, 3 joints
Links:
- removed link qolo_main
- added link tf_qolo, mass 50; collision mesh filename=package://qolo/../visualisation/urdf/stl/qolo_main.stl scale=1 1 1; visual mesh filename=package://qolo/../visualisation/urdf/stl/qolo_main.stl scale=1 1 1
- link bumper: geometry collision mesh filename=package://qolo/../visualisation/urdf/stl/bumper.stl scale=1 1 1; visual mesh filename=package://qolo/../visualisation/urdf/stl/bumper.stl scale=1 1 1
- link wheel_left: geometry collision mesh filename=package://qolo/../visualisation/urdf/stl/qolo_wheel.stl scale=1 1 1; visual mesh filename=package://qolo/../visualisation/urdf/stl/qolo_wheel.stl scale=1 1 1
- link wheel_right: geometry collision mesh filename=package://qolo/../visualisation/urdf/stl/qolo_wheel.stl scale=1 1 1; visual mesh filename=package://qolo/../visualisation/urdf/stl/qolo_wheel.stl scale=1 1 1
Joints:
- joint qolo_main_to_bumper: parent qolo_main -> tf_qolo
- joint qolo_main_to_wheel_left: parent qolo_main -> tf_qolo
- joint qolo_main_to_wheel_right: parent qolo_main -> tf_qolo

Commit message: + rviz bugfix

File: visualisation/urdf/qolo.urdf (robot description, URDF)
Before this commit: robot qolo, 4 links, 3 joints
Joints:
- joint qolo_main_to_wheel_left: type continuous -> fixed
- joint qolo_main_to_wheel_right: type continuous -> fixed
